File: Eagle/P4/PROTOTYPE4.brd (EAGLE design)
At the start: 38 x 66 mm, 14 parts, among them IC1 74HC00D, IC2 MS5611-01BA03, P12 TSW-112-02-S-S, P16 TSW-116-02-S-S, U1 AD8400AR1

Commit message: PROTOTYPE4 IN PROGRESS
Parts:
- removed P12: TSW-112-02-S-S, con-samtec:TSW-112-02-S-S
- removed P16: TSW-116-02-S-S, con-samtec:TSW-116-02-S-S
- added 0RX, 1TX, 3V3, A0, A1, A2, A3, A4, A5, BAT, D10, D11, D12, D13, D5, D6, D9, DFU, EN, EPD_3V3, EPD_BUSY, EPD_CS, EPD_DC, EPD_GND, EPD_MOSI, EPD_RST, EPD_SCK, GND, MISO, MOSI, REF, RST, SCK, SCL, SDA, USB: (no value), wirepad:SMD1,27-2,54
- moved R4 3.59 mm to (22.9, 17.8), turned to 270 degrees
- moved U$1 2.84 mm to (16.5, 63.5)
- moved Q1 2.84 mm to (22.9, 12.7), turned to 180 degrees
- moved LS1 1.27 mm to (31.8, 7.62)
- moved R1 1.27 mm to (24.1, 2.54)
- moved IC1 1.27 mm to (16.5, 6.35)
- moved S1 1.27 mm to (3.81, 6.35)
Connections:
- removed net 0RX: P16.3
- removed net 1TX: P16.2
- removed net A0: IC1.5, IC1.9, P16.12
- removed net A1: P16.11, R2.1, R3.2
- removed net A2: P16.10, U$1.2
- removed net A3: P16.9
- removed net A4: P16.8
- removed net A5: P16.7, U1.8
- removed net D10: P12.6
- removed net D11: P12.7
- removed net D12: P12.8
- removed net D13: P12.9
- removed net D5: P12.3
- removed net D6: P12.4
- removed net D9: P12.5
- removed net DFU: P16.1
- removed net N$4: C1.2, IC2.2, IC2.3
- removed net N$5: R3.1
- removed net N$8: U1.3
- removed net REF: P16.14
- removed net RST: P16.16
- removed net SCL: P12.2
- removed net SDA: P12.1
- removed net USB: P12.10
- removed net VCC: IC1.14
- new net BAT_MONITOR: D9.1
- new net BEEP_CTRL: A5.1, U1.8
- new net BUTTON_CTRL: A1.1, R2.1, R3.2
- new net EPD_BUSY: D12.1, EPD_BUSY.1
- new net EPD_CS: D6.1, EPD_CS.1
- new net EPD_DC: D10.1, EPD_DC.1
- new net EPD_RST: D11.1, EPD_RST.1
- new net MS5611_CSB: D13.1, IC2.4, IC2.5
- new net POT_CS: A3.1, U1.3
- new net PWR_CTRL: A0.1, IC1.5, IC1.9
- new net SD_CS: A2.1, U$1.2
- net 3V3: now also 3V3.1, C1.1, EPD_3V3.1, IC2.1; no longer P16.15
- net BAT: now also BAT.1, IC1.14; no longer P12.12
- net EN: now also EN.1; no longer P12.11
- net GND: now also C1.2, EPD_GND.1, GND.1, IC2.2, IC2.3; no longer P16.13
- net MISO: now also IC2.6, MISO.1; no longer P16.4
- net MOSI: now also EPD_MOSI.1, IC2.7, MOSI.1; no longer P16.5
- net N$3: now also IC1.8, R3.1; no longer C1.1, IC2.1
- net SCK: now also EPD_SCK.1, IC2.8, SCK.1; no longer P16.6
Routing:
- net GND: track 0.00 -> 118.8 mm, vias 0 -> 3
- net MOSI: track 0.00 -> 101.5 mm, vias 0 -> 2
- net 3V3: track 0.00 -> 74.1 mm, vias 0 -> 7
- net SCK: track 0.00 -> 73.6 mm, vias 0 -> 2
- net MISO: track 0.00 -> 49.2 mm
- net N$9: track 0.00 -> 42.6 mm
- net SD_CS: track 0.00 -> 38.6 mm
- net BAT: track 0.00 -> 31.2 mm
- net EPD_BUSY: track 0.00 -> 30.0 mm
- net POT_CS: track 0.00 -> 28.4 mm
- net MS5611_CSB: track 0.00 -> 28.0 mm, vias 0 -> 2
- net N$1: track 0.00 -> 25.6 mm, vias 0 -> 1
- net EN: track 0.00 -> 25.1 mm, vias 0 -> 4
- net EPD_DC: track 0.00 -> 25.0 mm
- net EPD_RST: track 0.00 -> 25.0 mm
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Other:
- board text added: "3V3"
- board text added: "BUSY"
- board text added: "CS"
- board text added: "DC"
- board text added: "GND"
- board text added: "MOSI"
- board text added: "PROTOTYPE[4]"
- board text added: "RST"
- board text added: "SCK"
- board text added: "v^SPEED VARIO"
