File: Eagle/P4/PROTOTYPE4.sch (EAGLE design)
At the start: 14 parts, among them IC1 74HC00D, IC2 MS5611-01BA03, P12 TSW-112-02-S-S, P16 TSW-116-02-S-S, U1 AD8400AR1

Commit message: PROTOTYPE4 IN PROGRESS
Parts:
- removed P12: TSW-112-02-S-S, con-samtec:TSW-112-02-S-S
- removed P16: TSW-116-02-S-S, con-samtec:TSW-116-02-S-S
- added 0RX, 1TX, 3V3, A0, A1, A2, A3, A4, A5, BAT, D10, D11, D12, D13, D5, D6, D9, DFU, EN, EPD_3V3, EPD_BUSY, EPD_CS, EPD_DC, EPD_GND, EPD_MOSI, EPD_RST, EPD_SCK, GND, MISO, MOSI, REF, RST, SCK, SCL, SDA, USB: (no value), wirepad:SMD2
Connections:
- removed net 0RX: P16-3.1
- removed net 1TX: P16-2.1
- removed net A0: IC1B.I1, IC1C.I0, P16-12.1
- removed net A1: P16-11.1, R2.1, R3.2
- removed net A2: P16-10.1, U$1.CS
- removed net A3: P16-9.1
- removed net A4: P16-8.1
- removed net A5: P16-7.1, U1.A1
- removed net D10: P12-6.1
- removed net D11: P12-7.1
- removed net D12: P12-8.1
- removed net D13: P12-9.1
- removed net D5: P12-3.1
- removed net D6: P12-4.1
- removed net D9: P12-5.1
- removed net DFU: P16-1.1
- removed net N$4: C1.2, IC2.GND, IC2.PS
- removed net N$5: R3.1
- removed net N$8: U1.CS*
- removed net REF: P16-14.1
- removed net RST: P16-16.1
- removed net SCL: P12-2.1
- removed net SDA: P12-1.1
- removed net USB: P12-10.1
- new net BAT_MONITOR: D9.P
- new net BEEP_CTRL: A5.P, U1.A1
- new net BUTTON_CTRL: A1.P, R2.1, R3.2
- new net EPD_BUSY: D12.P, EPD_BUSY.P
- new net EPD_CS: D6.P, EPD_CS.P
- new net EPD_DC: D10.P, EPD_DC.P
- new net EPD_RST: D11.P, EPD_RST.P
- new net MS5611_CSB: D13.P, IC2.CSB@1, IC2.CSB@2
- new net POT_CS: A3.P, U1.CS*
- new net PWR_CTRL: A0.P, IC1B.I1, IC1C.I0
- new net SD_CS: A2.P, U$1.CS
- net 3V3: now also 3V3.P, C1.1, EPD_3V3.P, IC2.VDD; no longer P16-15.1
- net BAT: now also BAT.P, IC1P.VCC; no longer P12-12.1
- net EN: now also EN.P; no longer P12-11.1
- net GND: now also C1.2, EPD_GND.P, GND.P, IC1P.GND, IC2.GND, IC2.PS; no longer P16-13.1
- net MISO: now also IC2.SDO, MISO.P; no longer P16-4.1
- net MOSI: now also EPD_MOSI.P, IC2.SDI/SDA, MOSI.P; no longer P16-5.1
- net N$3: now also IC1C.O, R3.1; no longer C1.1, IC2.VDD
- net SCK: now also EPD_SCK.P, IC2.SCLK, SCK.P; no longer P16-6.1
Other:
- note added: "2.9" E-PAPER DISPLAY"
- note added: "INTERNAL CONNECTION,"
- note added: "LEAVE OPEN------------>"
- moved on the sheet: C1, R2
