File: Eagle/P6_V3/Adafruit Feather Zero BLE rev B.brd (EAGLE design)
At the start: 68.4 x 25.3 mm, 55 parts, among them IC1 X9C102S, IC2 MS5611-01BA03, Q1 MMBT2222ALT3G, SW1 SPST_TACT-KMR2, U1 MBT40, U2 AP2112-3.3, U25 EVQP7A01P, U3 MCP73831T-2ACI/OT, U4 ATSAMD21G18_QFN, U41 EVQP7A01P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

Commit message: published app
Connections:
- removed net SWDCLK: X5.4
- net SWCLK: now also X5.4
Routing:
- net SWCLK: track 0.00 -> 14.6 mm
Changed lines of the file:
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@@
 <element name="IC2" library="Measurement-Specialties" package="SON125P300X500X100-8N" value="MS5611-01BA03" x="29.718" y="22.098" smashed="yes">
 <attribute name="MPN" value="MS5611-01BA03" x="29.718" y="22.098" size="1.778" layer="27" display="off"/>
+<attribute name="NAME" x="27.559" y="24.384" size="0.8128" layer="25" ratio="18"/>
 <attribute name="NAME" x="29.718" y="22.098" size="0.7" layer="51" ratio="5" rot="R90"/>
-<attribute name="NAME" x="27.559" y="24.384" size="0.8128" layer="25" ratio="18"/>
 <attribute name="VALUE" x="29.718" y="22.098" size="0.7" layer="27" ratio="5" rot="R90"/>
 </element>
@@
 <signal name="SWCLK">
 <contactref element="U4" pad="45"/>
+<contactref element="X5" pad="4"/>
+<wire x1="28.7776" y1="5.02106875" x2="28.76575" y2="4.936725" width="0.1524" layer="1"/>
+<wire x1="28.76575" y1="4.936725" x2="28.7776" y2="4.921" width="0.1524" layer="1"/>
+<wire x1="28.7776" y1="4.921" x2="28.7776" y2="4.67026875" width="0.1524" layer="1"/>
+<wire x1="28.7776" y1="4.67026875" x2="28.813596875" y2="4.634271875" width="0.1524" layer="1"/>
+<wire x1="28.813596875" y1="4.634271875" x2="28.829" y2="4.430625" width="0.1524" layer="1"/>
+<wire x1="28.829" y1="4.430625" x2="28.829" y2="4.28718125" width="0.1524" layer="1"/>
+<wire x1="39.48473125" y1="2.6206" x2="39.6484" y2="2.78426875" width="0.1524" layer="1"/>
+<wire x1="39.6484" y1="2.78426875" x2="39.6484" y2="3.5894" width="0.1524" layer="1"/>
+<wire x1="39.6484" y1="3.5894" x2="40.259" y2="4.2" width="0.1524" layer="1"/>
+<wire x1="28.682" y1="5.161" x2="28.76701875" y2="5.161" width="0.1524" layer="1"/>
+<wire x1="28.76701875" y1="5.161" x2="28.7776" y2="5.02106875" width="0.1524" layer="1"/>
+<wire x1="28.829" y1="4.28718125" x2="28.8788625" y2="3.62725" width="0.1524" layer="1"/>
+<wire x1="28.8788625" y1="3.62725" x2="29.8855125" y2="2.6206" width="0.1524" layer="1"/>
+<wire x1="29.8855125" y1="2.6206" x2="39.48473125" y2="2.6206" width="0.1524" layer="1"/>
 </signal>
 <signal name="SWDIO">
 <contactref element="U4" pad="46"/>
 <contactref element="X5" pad="2"/>
-<wire x1="29.165" y1="3.54" x2="29.165" y2="5.04" width="0.2032" layer="1"/>
-<wire x1="42.54" y1="3.54" x2="29.165" y2="3.54" width="0.2032" layer="16"/>
+<wire x1="29.927" y1="3.54" x2="29.927" y2="3.728" width="0.2032" layer="1"/>
+<wire x1="29.927" y1="3.728" x2="29.21" y2="4.445" width="0.2032" layer="1"/>
+<wire x1="29.21" y1="4.445" x2="29.165" y2="5.04" width="0.2032" layer="1"/>
+<wire x1="42.54" y1="3.54" x2="29.927" y2="3.54" width="0.2032" layer="16"/>
 <wire x1="41.54" y1="3.54" x2="42.54" y2="3.54" width="0.2032" layer="1"/>
 <wire x1="41.54" y1="4.165" x2="41.54" y2="3.54" width="0.2032" layer="1"/>
 <wire x1="29.165" y1="5.04" x2="29.182" y2="5.161" width="0.2032" layer="1"/>
 <wire x1="41.54" y1="4.165" x2="41.529" y2="4.2" width="0.2032" layer="1"/>
-<via x="29.165" y="3.54" extent="1-16" drill="0.3937"/>
+<via x="29.927" y="3.54" extent="1-16" drill="0.3937"/>
 <via x="42.54" y="3.54" extent="1-16" drill="0.3937"/>
 </signal>
@@
 <via x="45.29" y="11.79" extent="1-16" drill="0.3937"/>
 </signal>
-<signal name="SWDCLK">
-<contactref element="X5" pad="4"/>
-</signal>
 <signal name="A1_POT_INC">
