File: Eagle/P6_V4/Adafruit Feather Zero BLE rev B.brd (EAGLE design)
At the start: 68.4 x 25.3 mm, 59 parts, among them IC1 X9C102S, IC2 MS5611-01BA03, Q1 MMBT2222ALT3G, SW1 SPST_TACT-KMR2, U1 MBT40, U2 AP2112-3.3, U25 EVQP7A01P, U3 MCP73831T-2ACI/OT, U4 ATSAMD21G18_QFN, U41 EVQP7A01P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

Commit message: mini
Parts:
- removed U$26: (no value), adafruit:BLUEFRUITLOGO_100MM
- removed U$9: (no value), microbuilder:FEATHERLOGO
Other:
- board text removed: "3.7/4.2V LiPoly Batt µUSB charge"
- board text removed: "4 Reset,7 IRQ,8 CS"
- board text removed: "ATSAMD21G18 48MHz & 3.3V"
- board text removed: "Bluefruit Pins:"
- board text removed: "Feather M0 Bluefruit LE"
- board text removed: "SPI(SCK,MOSI,MISO)"
Changed lines of the file:
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@@
 <setting verticaltext="up"/>
 </settings>
-<grid distance="0.005" unitdist="inch" unit="mm" style="lines" multiple="1" display="no" altdistance="0.025" altunitdist="inch" altunit="inch"/>
+<grid distance="0.005" unitdist="inch" unit="inch" style="lines" multiple="1" display="no" altdistance="0.025" altunitdist="inch" altunit="inch"/>
 <layers>
 <layer number="1" name="Top" color="4" fill="1" visible="yes" active="yes"/>
@@
 <layer number="37" name="tTest" color="7" fill="1" visible="no" active="yes"/>
 <layer number="38" name="bTest" color="7" fill="1" visible="no" active="yes"/>
-<layer number="39" name="tKeepout" color="4" fill="11" visible="yes" active="yes"/>
-<layer number="40" name="bKeepout" color="1" fill="11" visible="yes" active="yes"/>
-<layer number="41" name="tRestrict" color="4" fill="10" visible="yes" active="yes"/>
-<layer number="42" name="bRestrict" color="1" fill="10" visible="yes" active="yes"/>
+<layer number="39" name="tKeepout" color="4" fill="11" visible="no" active="yes"/>
+<layer number="40" name="bKeepout" color="1" fill="11" visible="no" active="yes"/>
+<layer number="41" name="tRestrict" color="4" fill="10" visible="no" active="yes"/>
+<layer number="42" name="bRestrict" color="1" fill="10" visible="no" active="yes"/>
 <layer number="43" name="vRestrict" color="2" fill="10" visible="no" active="yes"/>
-<layer number="44" name="Drills" color="7" fill="1" visible="no" active="yes"/>
+<layer number="44" name="Drills" color="7" fill="1" visible="yes" active="yes"/>
 <layer number="45" name="Holes" color="7" fill="1" visible="yes" active="yes"/>
 <layer number="46" name="Milling" color="3" fill="1" visible="no" active="yes"/>
-<layer number="47" name="Measures" color="7" fill="1" visible="no" active="yes"/>
+<layer number="47" name="Measures" color="7" fill="1" visible="yes" active="yes"/>
 <layer number="48" name="Document" color="7" fill="1" visible="no" active="yes"/>
 <layer number="49" name="Reference" color="7" fill="1" visible="no" active="yes"/>
@@
 <text x="8.128" y="20.701" size="1.016" layer="21" ratio="12" rot="R270" align="center">#13</text>
 <text x="13.462" y="5.588" size="0.8128" layer="25" ratio="18" align="center">SW1</text>
-<text x="50.927" y="13.843" size="1.016" layer="22" font="vector" ratio="12" rot="SMR270" align="center">SPI(SCK,MOSI,MISO)</text>
-<text x="52.324" y="13.843" size="1.016" layer="22" font="vector" ratio="12" rot="SMR270" align="center">4 Reset,7 IRQ,8 CS</text>
-<text x="49.276" y="13.208" size="1.016" layer="22" font="vector" ratio="12" rot="SMR270" align="center">Bluefruit Pins:</text>
-<text x="11.43" y="22.987" size="1.016" layer="22" font="vector" ratio="13" rot="MR0" align="center">3.7/4.2V
-LiPoly Batt
-µUSB charge</text>
-<text x="28.956" y="18.542" size="1.27" layer="22" font="vector" ratio="13" rot="SMR0" align="center">Feather M0
-Bluefruit LE</text>
-<text x="42.418" y="20.32" size="1.143" layer="22" font="vector" ratio="15" rot="SMR0" align="center">ATSAMD21G18
-48MHz &amp; 3.3V</text>
 <dimension x1="0.127" y1="15.367" x2="50.8" y2="10.16" x3="25.4635" y3="30.607" textsize="1.778" layer="47" dtype="horizontal" unit="inch"/>
 <dimension x1="1.397" y1="2.413" x2="3.81" y2="2.413" x3="2.6035" y3="-3.429" textsize="1.778" layer="47" dtype="horizontal" unit="inch"/>
@@
 <wire x1="33.401" y1="13.97" x2="34.036" y2="13.97" width="0.2032" layer="21"/>
 <text x="32.639" y="14.351" size="1.016" layer="21" ratio="12" rot="R270" align="center">DFU</text>
+<wire x1="35.56" y1="14.97" x2="35.56" y2="12.97" width="0.1524" layer="22"/>
+<wire x1="36.56" y1="13.97" x2="34.56" y2="13.97" width="0.1524" layer="22"/>
+<wire x1="12.7" y1="23.495" x2="10.16" y2="23.495" width="0.1524" layer="22"/>
+<wire x1="10.16" y1="23.495" x2="10.16" y2="20.955" width="0.1524" layer="22"/>
+<wire x1="12.7" y1="4.445" x2="10.16" y2="4.445" width="0.1524" layer="22"/>
+<wire x1="10.16" y1="4.445" x2="10.16" y2="6.985" width="0.1524" layer="22"/>
+<wire x1="58.42" y1="23.495" x2="60.96" y2="23.495" width="0.1524" layer="22"/>
+<wire x1="60.96" y1="23.495" x2="60.96" y2="20.955" width="0.254" layer="22"/>
+<wire x1="58.42" y1="4.445" x2="60.96" y2="4.445" width="0.1524" layer="22"/>
+<wire x1="60.96" y1="4.445" x2="60.96" y2="6.985" width="0.1524" layer="22"/>
+<dimension x1="1.34" y1="5.08" x2="69.78" y2="5.08" x3="35.56" y3="-22.733" textsize="1.778" layer="47"/>
+<dimension x1="66.04" y1="26.6" x2="66.04" y2="1.34" x3="88.265" y3="13.97" textsize="1.778" layer="47"/>
 </plain>
 <attributes>
@@
 <attribute name="VALUE" x="32.512" y="22.987" size="0.8128" layer="27" font="vector" ratio="10" rot="R270"/>
 </element>
-<element name="U$26" library="adafruit" package="BLUEFRUITLOGO_100MM" value="" x="24.765" y="9.652" rot="MR0"/>
-<element name="U$9" library="microbuilder" package="FEATHERLOGO" value="" x="32.512" y="2.921" rot="MR0"/>
 <element name="IC2" library="Measurement-Specialties" package="SON125P300X500X100-8N" value="MS5611-01BA03" x="29.718" y="22.098" smashed="yes">
 <attribute name="MPN" value="MS5611-01BA03" x="29.718" y="22.098" size="1.778" layer="27" display="off"/>
